File: AD8129 Preamp Board.kicad_sch (KiCad schematic)
At the start: 35 parts, among them J1 Conn_01x03_Female, J2 Conn_Coaxial, J3 Conn_01x01_Female, T1 Transformer_1P_1S, U1 AD8129, U2 L78L06_SO8

Commit message: ADD(WIP): board layout
Parts:
- C1, C2, C3, C4, C5, C6, C7, C8, C9: footprint (none) -> AD8129 Preamp Board:C_0805_2012Metric
- D1, D2, D3, D4: footprint (none) -> AD8129 Preamp Board:D_SOD-323
- D5, D6, D7, D8: footprint (none) -> AD8129 Preamp Board:D_SOD-123
- J1: footprint (none) -> AD8129 Preamp Board:CONN-3
- R1, R2, R3, R4, R5, R6, R7, R8: footprint (none) -> AD8129 Preamp Board:R_0805_2012Metric
- U1: footprint (none) -> AD8129 Preamp Board:SOIC-8_3.9x4.9mm_P1.27mm
Other:
- note added: "Adjust R4, R5 for a desired Q, match within 0.1% or better."
- note added: "Match R3 to the antenna impedance."
- note added: "R4, R5 set gain Gain = 1 + Rf/Rg = = 1 + R7/R6"
- note removed: "Adjust R2, R3 for a desired Q, match within 0.1% or better."
- note removed: "Match R1 to the antenna impedance."
- note removed: "R4, R5 set gain Gain = 1 + Rf/Rg = = 1 + R5/R4"

Commit message: FIX: restore after crash
Parts:
- L1, L2, L4: footprint (none) -> AD8129 Preamp Board:L_1812_4532Metric_Pad1.30x3.40mm_HandSolder
Changed lines of the file:
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@@
       (effects (font (size 1.27 1.27)) (justify left))
     )
-    (property "Footprint" "" (id 2) (at 228.6 69.215 0)
+    (property "Footprint" "AD8129 Preamp Board:L_1812_4532Metric_Pad1.30x3.40mm_HandSolder" (id 2) (at 228.6 69.215 0)
       (effects (font (size 1.27 1.27)) hide)
     )
@@
     (property "Reference" "L1" (id 0) (at 152.4 37.465 90))
     (property "Value" "220uH" (id 1) (at 152.4 40.005 90))
-    (property "Footprint" "" (id 2) (at 152.4 43.815 0)
+    (property "Footprint" "AD8129 Preamp Board:L_1812_4532Metric_Pad1.30x3.40mm_HandSolder" (id 2) (at 152.4 43.815 0)
       (effects (font (size 1.27 1.27)) hide)
     )
@@
     (property "Reference" "L2" (id 0) (at 152.4 120.015 90))
     (property "Value" "220uH" (id 1) (at 152.4 122.555 90))
-    (property "Footprint" "" (id 2) (at 152.4 125.095 0)
+    (property "Footprint" "AD8129 Preamp Board:L_1812_4532Metric_Pad1.30x3.40mm_HandSolder" (id 2) (at 152.4 125.095 0)
       (effects (font (size 1.27 1.27)) hide)
     )
@@
     )
     (path "/7735ef7e-0d05-4ae5-b498-7db60adee0e6"
-      (reference "L1") (unit 1) (value "220uH") (footprint "")
+      (reference "L1") (unit 1) (value "220uH") (footprint "AD8129 Preamp Board:L_1812_4532Metric_Pad1.30x3.40mm_HandSolder")
     )
     (path "/b6864b4f-d329-4382-9e55-67de1bf05f05"
-      (reference "L2") (unit 1) (value "220uH") (footprint "")
+      (reference "L2") (unit 1) (value "220uH") (footprint "AD8129 Preamp Board:L_1812_4532Metric_Pad1.30x3.40mm_HandSolder")
     )
     (path "/8146b11a-fccb-48a7-bcaa-9e1b77e1c86b"
@@
     )
     (path "/4886c859-4e3e-44ea-8304-93581e52b72f"
-      (reference "L4") (unit 1) (value "220uH") (footprint "")
+      (reference "L4") (unit 1) (value "220uH") (footprint "AD8129 Preamp Board:L_1812_4532Metric_Pad1.30x3.40mm_HandSolder")
     )
     (path "/827c9052-7417-4998-8820-0ee4048dfc60"

Commit message: FIX: pass ERC
Parts:
- J1: value Conn_01x03_Female -> ANT
- J2: renamed from J3; value Conn_01x01_Female -> TUNE
- J3: renamed from J2; value Conn_Coaxial -> TRX
Other:
- moved on the sheet: C1, C2, C3, C4, C5, C6, C7, C8, C9, D1, D2, D3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

Commit message: ADD: board name, revision, date. Board verified.
Other:
- title: (none) -> AD8129 Preamp Board
Changed lines of the file:
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@@
 (kicad_sch (version 20211123) (generator eeschema)
   (paper "A4")
+  (title_block
+    (title "AD8129 Preamp Board")
+    (date "2022-07-06")
+    (rev "1")
+  )
   (junction (at 73.025 116.84) (diameter 0) (color 0 0 0 0)
   )

Commit message: FIX: silkscreen line width
Parts:
- J1: footprint AD8129 Preamp Board:CONN-3 -> AD8129 Preamp Board:WirePad_3_0.8_1.5
- J2: footprint (none) -> AD8129 Preamp Board:WirePad_1_0.8_1.5
- L3: footprint (none) -> AD8129 Preamp Board:L_1812_4532Metric_Pad1.30x3.40mm_HandSolder
Changed lines of the file:
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@@
   (symbol (lib_id "power:PWR_FLAG") (at 229.87 53.34 0) (unit 1)
     (in_bom yes) (on_board yes) (fields_autoplaced)
-    (property "Reference" "#FLG0103" (id 0) (at 229.87 51.435 0)
+    (property "Reference" "#FLG04" (id 0) (at 229.87 51.435 0)
       (effects (font (size 1.27 1.27)) hide)
     )
@@
     (property "Reference" "J1" (id 0) (at 41.275 76.2 0))
     (property "Value" "ANT" (id 1) (at 41.275 78.74 0))
-    (property "Footprint" "AD8129 Preamp Board:CONN-3" (id 2) (at 40.64 83.82 0)
+    (property "Footprint" "AD8129 Preamp Board:WirePad_3_0.8_1.5" (id 2) (at 40.64 83.82 0)
       (effects (font (size 1.27 1.27)) hide)
     )
@@
   (symbol (lib_id "power:PWR_FLAG") (at 147.32 139.7 180) (unit 1)
     (in_bom yes) (on_board yes) (fields_autoplaced)
-    (property "Reference" "#FLG0101" (id 0) (at 147.32 141.605 0)
+    (property "Reference" "#FLG01" (id 0) (at 147.32 141.605 0)
       (effects (font (size 1.27 1.27)) hide)
     )
@@
       (effects (font (size 1.27 1.27)) (justify left))
     )
-    (property "Footprint" "" (id 2) (at 223.52 81.28 0)
+    (property "Footprint" "AD8129 Preamp Board:L_1812_4532Metric_Pad1.30x3.40mm_HandSolder" (id 2) (at 223.52 81.28 0)
       (effects (font (size 1.27 1.27)) hide)
     )
@@
   (symbol (lib_id "power:PWR_FLAG") (at 149.86 74.93 0) (unit 1)
     (in_bom yes) (on_board yes) (fields_autoplaced)
-    (property "Reference" "#FLG0102" (id 0) (at 149.86 73.025 0)
+    (property "Reference" "#FLG02" (id 0) (at 149.86 73.025 0)
       (effects (font (size 1.27 1.27)) hide)
     )
@@
   (symbol (lib_id "power:PWR_FLAG") (at 208.28 77.47 180) (unit 1)
     (in_bom yes) (on_board yes) (fields_autoplaced)
-    (property "Reference" "#FLG0104" (id 0) (at 208.28 79.375 0)
+    (property "Reference" "#FLG03" (id 0) (at 208.28 79.375 0)
       (effects (font (size 1.27 1.27)) hide)
     )
@@
       (effects (font (size 1.27 1.27)) (justify left))
     )
-    (property "Footprint" "" (id 2) (at 236.22 110.49 0)
+    (property "Footprint" "AD8129 Preamp Board:WirePad_1_0.8_1.5" (id 2) (at 236.22 110.49 0)
       (effects (font (size 1.27 1.27)) hide)
     )
@@
   (symbol_instances
     (path "/7cdeac05-e4be-462c-8716-03765a1d8065"
-      (reference "#FLG0101") (unit 1) (value "PWR_FLAG") (footprint "")
+      (reference "#FLG01") (unit 1) (value "PWR_FLAG") (footprint "")
     )
     (path "/acd7bd34-0f26-4375-82af-9fc9101d2bb8"
-      (reference "#FLG0102") (unit 1) (value "PWR_FLAG") (footprint "")
+      (reference "#FLG02") (unit 1) (value "PWR_FLAG") (footprint "")
+    )
+    (path "/d66c5b4c-fcad-46bc-9a52-789856b29f0b"
+      (reference "#FLG03") (unit 1) (value "PWR_FLAG") (footprint "")
     )
     (path "/070fb985-d30c-4781-a72a-a90cb6950444"
-      (reference "#FLG0103") (unit 1) (value "PWR_FLAG") (footprint "")
-    )
-    (path "/d66c5b4c-fcad-46bc-9a52-789856b29f0b"
-      (reference "#FLG0104") (unit 1) (value "PWR_FLAG") (footprint "")
+      (reference "#FLG04") (unit 1) (value "PWR_FLAG") (footprint "")
     )
     (path "/c7ae8597-5a59-42cd-8bba-a46955e5aefc"
@@
     )
     (path "/0a2d9ea1-26b2-42a6-bbbe-a3f042fb6f34"
-      (reference "J1") (unit 1) (value "ANT") (footprint "AD8129 Preamp Board:CONN-3")
+      (reference "J1") (unit 1) (value "ANT") (footprint "AD8129 Preamp Board:WirePad_3_0.8_1.5")
     )
     (path "/e931ab96-5377-4628-8122-7934ffab892c"
-      (reference "J2") (unit 1) (value "TUNE") (footprint "")
+      (reference "J2") (unit 1) (value "TUNE") (footprint "AD8129 Preamp Board:WirePad_1_0.8_1.5")
     )
     (path "/45c4b5cd-ee34-40a1-ad17-465c5c808423"
@@
     )
     (path "/8146b11a-fccb-48a7-bcaa-9e1b77e1c86b"
-      (reference "L3") (unit 1) (value "1mH") (footprint "")
+      (reference "L3") (unit 1) (value "1mH") (footprint "AD8129 Preamp Board:L_1812_4532Metric_Pad1.30x3.40mm_HandSolder")
     )
     (path "/4886c859-4e3e-44ea-8304-93581e52b72f"

Commit message: ADD: all footprints
Parts:
- J3: footprint (none) -> AD8129 Preamp Board:SMA_Samtec_SMA-J-P-X-ST-EM1_EdgeMount
- T1: footprint (none) -> AD8129 Preamp Board:TR-FT-50-43-1P-1S-Isolated
Changed lines of the file:
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@@
       (effects (font (size 1.27 1.27)) (justify left))
     )
-    (property "Footprint" "" (id 2) (at 242.57 90.17 0)
+    (property "Footprint" "AD8129 Preamp Board:SMA_Samtec_SMA-J-P-X-ST-EM1_EdgeMount" (id 2) (at 242.57 90.17 0)
       (effects (font (size 1.27 1.27)) hide)
     )
@@
     (property "Reference" "T1" (id 0) (at 184.1627 85.09 0))
     (property "Value" "Transformer_1P_1S" (id 1) (at 184.1627 87.63 0))
-    (property "Footprint" "" (id 2) (at 184.15 95.25 0)
+    (property "Footprint" "AD8129 Preamp Board:TR-FT-50-43-1P-1S-Isolated" (id 2) (at 184.15 95.25 0)
       (effects (font (size 1.27 1.27)) hide)
     )
@@
     )
     (path "/45c4b5cd-ee34-40a1-ad17-465c5c808423"
-      (reference "J3") (unit 1) (value "TRX") (footprint "")
+      (reference "J3") (unit 1) (value "TRX") (footprint "AD8129 Preamp Board:SMA_Samtec_SMA-J-P-X-ST-EM1_EdgeMount")
     )
     (path "/7735ef7e-0d05-4ae5-b498-7db60adee0e6"
@@
     )
     (path "/f7ad2744-8981-4b98-a696-86b5a0e44036"
-      (reference "T1") (unit 1) (value "Transformer_1P_1S") (footprint "")
+      (reference "T1") (unit 1) (value "Transformer_1P_1S") (footprint "AD8129 Preamp Board:TR-FT-50-43-1P-1S-Isolated")
     )
     (path "/23ca2cb0-3422-4d12-ac8b-2c3f9709b23a"

Commit message: ADD: pcb layout, needs via stitching
Parts:
- added H1, H2, H3, H4: M3, AD8129 Preamp Board:MountingHole_3.2mm_M3, symbol AD8129 Preamp Board:MountingHole
Connections:
- net REGGND: now reaches C7.2, C9.2, L2.1, L3.1, U2.2 (GND), U2.3 (GND), U2.6 (GND), U2.7 (GND)
Other:
- note added: "Mounting Holes"
Changed lines of the file:
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@@
   (junction (at 63.5 83.82) (diameter 0) (color 0 0 0 0)
   )
+  (junction (at 203.2 78.74) (diameter 0) (color 0 0 0 0)
+  )
   (junction (at 223.52 62.23) (diameter 0) (color 0 0 0 0)
   )
@@
     (stroke (width 0) (type default) (color 0 0 0 0))
   )
+  (polyline (pts (xy 83.82 166.37) (xy 83.82 144.78))
+    (stroke (width 0) (type default) (color 0 0 0 0))
+  )
   (wire (pts (xy 157.48 55.88) (xy 229.87 55.88))
     (stroke (width 0) (type default) (color 0 0 0 0))
@@
     (stroke (width 0) (type default) (color 0 0 0 0))
   )
+  (polyline (pts (xy 57.15 144.78) (xy 83.82 144.78))
+    (stroke (width 0) (type default) (color 0 0 0 0))
+  )
   (wire (pts (xy 72.39 93.98) (xy 72.39 95.25))
     (stroke (width 0) (type default) (color 0 0 0 0))
@@
     (stroke (width 0) (type default) (color 0 0 0 0))
   )
+  (polyline (pts (xy 57.15 144.78) (xy 57.15 166.37))
+    (stroke (width 0) (type default) (color 0 0 0 0))
+  )
   (wire (pts (xy 111.76 106.68) (xy 111.76 109.22))
     (stroke (width 0) (type default) (color 0 0 0 0))
@@
     (stroke (width 0) (type default) (color 0 0 0 0))
   )
-  (wire (pts (xy 203.2 74.93) (xy 203.2 137.16))
+  (wire (pts (xy 203.2 74.93) (xy 203.2 78.74))
     (stroke (width 0) (type default) (color 0 0 0 0))
   )
@@
     (stroke (width 0) (type default) (color 0 0 0 0))
   )
+  (wire (pts (xy 203.2 78.74) (xy 203.2 137.16))
+    (stroke (width 0) (type default) (color 0 0 0 0))
+  )
   (wire (pts (xy 198.12 100.33) (xy 212.09 100.33))
     (stroke (width 0) (type default) (color 0 0 0 0))
@@
     (stroke (width 0) (type default) (color 0 0 0 0))
   )
+  (wire (pts (xy 200.66 78.74) (xy 203.2 78.74))
+    (stroke (width 0) (type default) (color 0 0 0 0))
+  )
   (wire (pts (xy 143.51 66.04) (xy 146.05 66.04))
     (stroke (width 0) (type default) (color 0 0 0 0))
   )
   (wire (pts (xy 147.32 66.04) (xy 147.32 55.88))
+    (stroke (width 0) (type default) (color 0 0 0 0))
+  )
+  (polyline (pts (xy 57.15 166.37) (xy 83.82 166.37))
     (stroke (width 0) (type default) (color 0 0 0 0))
   )
@@
   (text "Adjust R4, R5 for\na desired Q, match\nwithin 0.1% or better.\n"
     (at 114.935 60.325 0)
+    (effects (font (size 1.27 1.27)) (justify left bottom))
+  )
+  (text "Mounting Holes" (at 58.42 165.1 0)
     (effects (font (size 1.27 1.27)) (justify left bottom))
   )
@@
     (property "Intersheet References" "${INTERSHEET_REFS}" (id 0) (at 82.1812 127.7144 0)
       (effects (font (size 1.27 1.27)) (justify left) hide)
+    )
+  )
+  (global_label "REGGND" (shape input) (at 200.66 78.74 180) (fields_autoplaced)
+    (effects (font (size 1.27 1.27)) (justify right))
+    (property "Intersheet References" "${INTERSHEET_REFS}" (id 0) (at 190.6874 78.6606 0)
+      (effects (font (size 1.27 1.27)) (justify right) hide)
     )
   )
@@
     (pin "8")
   )
+  (symbol (lib_id "AD8129 Preamp Board:MountingHole") (at 74.93 148.59 0) (unit 1)
+    (in_bom no) (on_board yes) (fields_autoplaced)
+    (property "Reference" "H3" (id 0) (at 77.47 147.3199 0)
+      (effects (font (size 1.27 1.27)) (justify left))
+    )
+    (property "Value" "M3" (id 1) (at 77.47 149.8599 0)
+      (effects (font (size 1.27 1.27)) (justify left))
+    )
+    (property "Footprint" "AD8129 Preamp Board:MountingHole_3.2mm_M3" (id 2) (at 74.93 148.59 0)
+      (effects (font (size 1.27 1.27)) hide)
+    )
+    (property "Datasheet" "~" (id 3) (at 74.93 148.59 0)
+      (effects (font (size 1.27 1.27)) hide)
+    )
+  )
   (symbol (lib_id "power:PWR_FLAG") (at 229.87 53.34 0) (unit 1)
     (in_bom yes) (on_board yes) (fields_autoplaced)
@@
     (pin "2")
     (pin "3")
+  )
+  (symbol (lib_id "AD8129 Preamp Board:MountingHole") (at 60.96 157.48 0) (unit 1)
+    (in_bom yes) (on_board yes) (fields_autoplaced)
+    (property "Reference" "H2" (id 0) (at 63.5 156.2099 0)
+      (effects (font (size 1.27 1.27)) (justify left))
+    )
+    (property "Value" "M3" (id 1) (at 63.5 158.7499 0)
+      (effects (font (size 1.27 1.27)) (justify left))
+    )
+    (property "Footprint" "AD8129 Preamp Board:MountingHole_3.2mm_M3" (id 2) (at 60.96 157.48 0)
+      (effects (font (size 1.27 1.27)) hide)
+    )
+    (property "Datasheet" "~" (id 3) (at 60.96 157.48 0)
+      (effects (font (size 1.27 1.27)) hide)
+    )
   )
   (symbol (lib_id "AD8129 Preamp Board:AD8129") (at 146.05 90.17 0) (unit 1)
@@
     (pin "1")
   )
+  (symbol (lib_id "AD8129 Preamp Board:MountingHole") (at 74.93 157.48 0) (unit 1)
+    (in_bom no) (on_board yes) (fields_autoplaced)
+    (property "Reference" "H4" (id 0) (at 77.47 156.2099 0)
+      (effects (font (size 1.27 1.27)) (justify left))
+    )
+    (property "Value" "M3" (id 1) (at 77.47 158.7499 0)
+      (effects (font (size 1.27 1.27)) (justify left))
+    )
+    (property "Footprint" "AD8129 Preamp Board:MountingHole_3.2mm_M3" (id 2) (at 74.93 157.48 0)
+      (effects (font (size 1.27 1.27)) hide)
+    )
+    (property "Datasheet" "~" (id 3) (at 74.93 157.48 0)
+      (effects (font (size 1.27 1.27)) hide)
+    )
+  )
   (symbol (lib_id "power:GND") (at 133.35 127 270) (unit 1)
     (in_bom yes) (on_board yes) (fields_autoplaced)
@@
     (pin "2")
   )
+  (symbol (lib_id "AD8129 Preamp Board:MountingHole") (at 60.96 148.59 0) (unit 1)
+    (in_bom no) (on_board yes) (fields_autoplaced)
+    (property "Reference" "H1" (id 0) (at 63.5 147.3199 0)
+      (effects (font (size 1.27 1.27)) (justify left))
+    )
+    (property "Value" "M3" (id 1) (at 63.5 149.8599 0)
+      (effects (font (size 1.27 1.27)) (justify left))
+    )
+    (property "Footprint" "AD8129 Preamp Board:MountingHole_3.2mm_M3" (id 2) (at 60.96 148.59 0)
+      (effects (font (size 1.27 1.27)) hide)
+    )
+    (property "Datasheet" "~" (id 3) (at 60.96 148.59 0)
+      (effects (font (size 1.27 1.27)) hide)
+    )
+  )
   (symbol (lib_id "AD8129 Preamp Board:R") (at 133.35 111.76 0) (unit 1)
     (in_bom yes) (on_board yes) (fields_autoplaced)
@@
       (reference "D8") (unit 1) (value "1N4148W") (footprint "AD8129 Preamp Board:D_SOD-123")
     )
+    (path "/ba03f6c8-7183-433f-9763-ab78111ee96e"
+      (reference "H1") (unit 1) (value "M3") (footprint "AD8129 Preamp Board:MountingHole_3.2mm_M3")
+    )
+    (path "/10768a52-fff1-470b-9fd0-4f907b43be9b"
+      (reference "H2") (unit 1) (value "M3") (footprint "AD8129 Preamp Board:MountingHole_3.2mm_M3")
+    )
+    (path "/06717f15-493b-49d6-842a-aa6c3b44560e"
+      (reference "H3") (unit 1) (value "M3") (footprint "AD8129 Preamp Board:MountingHole_3.2mm_M3")
+    )
+    (path "/6483a9db-ec5c-4c23-86cf-17c6b637c8b8"
+      (reference "H4") (unit 1) (value "M3") (footprint "AD8129 Preamp Board:MountingHole_3.2mm_M3")
+    )
     (path "/0a2d9ea1-26b2-42a6-bbbe-a3f042fb6f34"

Commit message: ADD: v1 final touch
Other:
- note added: "Adjust R4, R5 for a desired Q, match within 0.1%."
- note added: "R7, R6 set gain Gain = 1 + Rf/Rg = = 1 + R7/R6"
- note removed: "Adjust R4, R5 for a desired Q, match within 0.1% or better."
- note removed: "R4, R5 set gain Gain = 1 + Rf/Rg = = 1 + R7/R6"
Changed lines of the file:
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@@
     (stroke (width 0) (type default) (color 0 0 0 0))
   )
-  (text "Adjust R4, R5 for\na desired Q, match\nwithin 0.1% or better.\n"
+  (text "Adjust R4, R5 for\na desired Q, match\nwithin 0.1%.\n"
     (at 114.935 60.325 0)
     (effects (font (size 1.27 1.27)) (justify left bottom))
@@
     (effects (font (size 1.27 1.27)) (justify left bottom))
   )
-  (text "R4, R5 set gain\nGain = 1 + Rf/Rg =\n= 1 + R7/R6" (at 147.32 116.205 0)
+  (text "R7, R6 set gain\nGain = 1 + Rf/Rg =\n= 1 + R7/R6" (at 147.32 116.205 0)
     (effects (font (size 1.27 1.27)) (justify left bottom))
   )
