File: AD8129 Preamp Board.kicad_sch (KiCad schematic)
At the start: 39 parts, among them J1 ANT, J2 TUNE, J3 TRX, T1 Transformer_1P_1S, U1 AD8129, U2 L78L06_SO8

Commit message: FIX: schematics name and date
Other:
- title: AD8129 Preamp Board -> AD8129 RX Antenna Amp
Changed lines of the file:
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@@
   (paper "A4")
   (title_block
-    (title "AD8129 Preamp Board")
-    (date "2022-07-06")
+    (title "AD8129 RX Antenna Amp")
+    (date "2022-07-07")
     (rev "1")
   )

Commit message: ADD: capacitors, T1 shield
Parts:
- added C2, C4, C5, C8: 100n, AD8129 Preamp Board:C_0805_2012Metric, symbol AD8129 Preamp Board:C
- renumbered C6 to C10, C7 to C11, C8 to C12, C9 to C13, C2 to C3, C3 to C6, C4 to C7, C5 to C9
Connections:
- net GND: now also C2.2, C4.2, C5.1, C8.2
- net at C10.2, C7.1, L2.2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: now also C8.1
- net at C6.2, C9.1, L1.1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: now also C5.2
- net at D1.1 (K), D2.1 (K), D3.1 (K)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: now also C2.1, C4.1
Other:
- moved on the sheet: C1, C3, H1, H2, H3, H4, J1, L1, L2, R1, R2
