File: ad8129-rx-antenna-amp.kicad_sch (KiCad schematic)
At the start: 43 parts, among them J1 ANT, J2 TUNE, J3 TRX, T1 Transformer_1P_1S, U1 AD8129, U2 L78L06_SO8

Commit message: FIX: change project file names to match GitHub project name
Parts:
- C1, C10, C11, C12, C13, C2, C3, C4, C5, C6, C7, C8, C9: footprint AD8129 Preamp Board:C_0805_2012Metric -> ad8129-rx-antenna-amp:C_0805_2012Metric; symbol AD8129 Preamp Board:C -> ad8129-rx-antenna-amp:C
- D1, D2, D3, D4: footprint AD8129 Preamp Board:D_SOD-323 -> ad8129-rx-antenna-amp:D_SOD-323; symbol AD8129 Preamp Board:VD -> ad8129-rx-antenna-amp:VD
- D5, D6, D7, D8: footprint AD8129 Preamp Board:D_SOD-123 -> ad8129-rx-antenna-amp:D_SOD-123; symbol AD8129 Preamp Board:D -> ad8129-rx-antenna-amp:D
- H1, H2, H3, H4: footprint AD8129 Preamp Board:MountingHole_3.2mm_M3 -> ad8129-rx-antenna-amp:MountingHole_3.2mm_M3; symbol AD8129 Preamp Board:MountingHole -> ad8129-rx-antenna-amp:MountingHole
- J1: footprint AD8129 Preamp Board:WirePad_3_0.8_1.5 -> ad8129-rx-antenna-amp:WirePad_3_0.8_1.5; symbol AD8129 Preamp Board:Conn_01x03_Female -> ad8129-rx-antenna-amp:Conn_01x03_Female
- J2: footprint AD8129 Preamp Board:WirePad_1_0.8_1.5 -> ad8129-rx-antenna-amp:WirePad_1_0.8_1.5; symbol AD8129 Preamp Board:Conn_01x01_Female -> ad8129-rx-antenna-amp:Conn_01x01_Female
- J3: footprint AD8129 Preamp Board:SMA_Samtec_SMA-J-P-X-ST-EM1_EdgeMount -> ad8129-rx-antenna-amp:SMA_Samtec_SMA-J-P-X-ST-EM1_EdgeMount; symbol AD8129 Preamp Board:Conn_Coaxial -> ad8129-rx-antenna-amp:Conn_Coaxial
- L1, L2, L3, L4: footprint AD8129 Preamp Board:L_1812_4532Metric_Pad1.30x3.40mm_HandSolder -> ad8129-rx-antenna-amp:L_1812_4532Metric_Pad1.30x3.40mm_HandSolder; symbol AD8129 Preamp Board:L -> ad8129-rx-antenna-amp:L
- R1, R2, R3, R4, R5, R6, R7, R8: footprint AD8129 Preamp Board:R_0805_2012Metric -> ad8129-rx-antenna-amp:R_0805_2012Metric; symbol AD8129 Preamp Board:R -> ad8129-rx-antenna-amp:R
- T1: footprint AD8129 Preamp Board:TR-FT-50-43-1P-1S-Isolated -> ad8129-rx-antenna-amp:TR-FT-50-43-1P-1S-Isolated; symbol AD8129 Preamp Board:Transformer_1P_1S -> ad8129-rx-antenna-amp:Transformer_1P_1S
- U1: footprint AD8129 Preamp Board:SOIC-8_3.9x4.9mm_P1.27mm -> ad8129-rx-antenna-amp:SOIC-8_3.9x4.9mm_P1.27mm; symbol AD8129 Preamp Board:AD8129 -> ad8129-rx-antenna-amp:AD8129
- U2: symbol AD8129 Preamp Board:L78L06_SO8 -> ad8129-rx-antenna-amp:L78L06_SO8
